Commit message: Change param navigation

File: turtlebot3_description/urdf/mybot.xacro (robot description, xacro)
@@ -290,4 +290,10 @@
     </collision>
   </link>
+    <joint name="imu_joint" type="fixed">
+    <parent link="base_link"/>
+    <child link="imu_link"/>
+    <origin xyz="0 0 0" rpy="0 0 0"/>
+  </joint>
+  <link name="imu_link"/>
   <joint
     name="lidar_joint"

Commit message: Change RPlidar a2m8 to sick tim240
Change /laser frame to /cloud frame.
Sick tim240 publish both /scan and /cloud topic.

File: turtlebot3_description/urdf/mybot.xacro (robot description, xacro)
@@ -4,11 +4,15 @@
   <xacro:include filename="$(find service_robot)/urdf/materials.xacro" />
   <xacro:include filename="$(find service_robot)/urdf/macros.xacro" />
+  <link name="base_footprint"/>
+  <joint name="base_joint" type="fixed">
+    <parent link="base_footprint"/>
+    <child link="base_link"/>
+    <origin xyz="0.0 0.0 0.010" rpy="0 0 0"/>
+  </joint>
   <link name="base_link">
     <inertial>
-      <origin
-        xyz="0.000508426452289656 5.85230715788032E-05 0.532734267230434"
-        rpy="0 0 0" />
+      <origin xyz="0 0 0" rpy="0 0 0"/>
       <mass
-        value="56.8425142723701" />
+        value="8.2573504e-01" />
       <inertia
         ixx="4.9887479320299"
@@ -251,5 +255,5 @@
   </joint>
   <link
-    name="laser">
+    name="cloud">
     <inertial>
       <origin
@@ -305,5 +309,5 @@
       link="base_link" />
     <child
-      link="laser" />
+      link="cloud" />
     <axis
       xyz="0 0 0" />

Commit message: backup

File: turtlebot3_description/urdf/mybot.xacro (robot description, xacro)
@@ -8,11 +8,29 @@
     <parent link="base_footprint"/>
     <child link="base_link"/>
-    <origin xyz="0.0 0.0 0.010" rpy="0 0 0"/>
-  </joint>
+    <origin xyz="0.0 0.0 0.0" rpy="0 0 0"/>
+  </joint>
+  <!-- Begin base_link -->
   <link name="base_link">
+    <visual>
+      <origin
+        xyz="0 0 0" rpy="0 0 0" />
+      <geometry>
+        <mesh filename="package://service_robot/meshes/base_link.STL" />
+      </geometry>
+      <material name="">
+        <color rgba="0.647058823529412 0.619607843137255 0.588235294117647 1" />
+      </material>
+    </visual>
+    <collision>
+      <origin
+        xyz="0 0 0"
+        rpy="0 0 0" />
+      <geometry>
+      <mesh filename="package://service_robot/meshes/base_link.STL" />
+      </geometry>
+    </collision>
     <inertial>
       <origin xyz="0 0 0" rpy="0 0 0"/>
-      <mass
-        value="8.2573504e-01" />
+      <mass value="42.124" />
       <inertia
         ixx="4.9887479320299"
@@ -23,123 +41,78 @@
         izz="2.8376872224854" />
     </inertial>
-    <visual>
-      <origin
-        xyz="0 0 0"
-        rpy="0 0 0" />
-      <geometry>
-        <mesh
-          filename="package://service_robot/meshes/base_link.STL" />
-      </geometry>
-      <material
-        name="">
+  </link>
+  <!-- End base_link -->
+  <!-- Connect base_link to wheel_left_link by wheel_left_joint-->
+  <joint name="wheel_left_joint" type="continuous">
+    <parent link="base_link" />
+    <child link="wheel_left_link" />
+    <origin xyz="0.0047501 0.241 0.073998" rpy="0 0 0" />
+    <axis xyz="0 1 0" />
+  </joint>
+  <!-- Begin wheel_left_link -->
+ <link name="wheel_left_link">
+     <visual>
+      <origin xyz="0 0 0" rpy="0 0 0"/>
+      <geometry>
+        <mesh filename="package://service_robot/meshes/wheel_left_link.STL" />
+      </geometry>
+      <material name="">
+        <color rgba="0 0 0 1" />
+      </material>
+    </visual>
+    <collision>
+      <origin xyz="0 0 0" rpy="0 0 0" />
+      <geometry>
+      <mesh filename="package://service_robot/meshes/wheel_left_link.STL" />
+      </geometry>
+    </collision>
+    <inertial>
+      <origin
+        xyz="0 0 0"
+        rpy="0 0 0" />
+      <mass
+        value="0.238183102723088" />
+      <inertia
+        ixx="0.000429468568590385"
+        ixy="2.82194133801453E-08"
+        ixz="3.45307405175469E-09"
+        iyy="0.000813895351440581"
+        iyz="9.00820636504668E-09"
+        izz="0.000429448713932949" />
+    </inertial>
+  </link>
+<!-- End wheel_left_link -->
+   <!-- Connect base_link to wheel_right_link by wheel_right_joint-->
+  <joint
+    name="wheel_right_joint" type="continuous">
+    <parent link="base_link" />
+    <child link="wheel_right_link" />
+    <origin	xyz="0.0049293 -0.235 0.0740" rpy="0 0 0" />
+    <axis xyz="0 1 0" />
+  </joint>
+<!-- Begin wheel_right_link -->
+ <link name="wheel_right_link">
+     <visual>
+      <origin
+        xyz="0 0 0" rpy="0 0 0" />
+      <geometry>
+        <mesh filename="package://service_robot/meshes/wheel_right_link.STL" />
+      </geometry>
+      <material name="">
         <color
-          rgba="0.647058823529412 0.619607843137255 0.588235294117647 1" />
-      </material>
-    </visual>
-    <collision>
-      <origin
-        xyz="0 0 0"
-        rpy="0 0 0" />
-      <geometry>
-        <mesh
-          filename="package://service_robot/meshes/base_link.STL" />
-      </geometry>
-    </collision>
-    <collision name='caster_1_collision'>
-      <origin xyz="0.165 0.09 0.031" rpy=" 0 0 0"/>
-      <geometry>
-        <sphere radius="0.03"/>
-      </geometry>
-      <surface>
-        <friction>
-          <ode>
-            <mu>0</mu>
-            <mu2>0</mu2>
-            <slip1>1.0</slip1>
-            <slip2>1.0</slip2>
-          </ode>
-        </friction>
-      </surface>
-    </collision>
-    <visual name='caster_1_visual'>
-      <origin xyz="0.165 0.09 0.031" rpy=" 0 0 0"/>
-      <geometry>
-        <sphere radius="0.03"/>
-      </geometry>
-    </visual>
-    <collision name='caster_2_collision'>
-      <origin xyz="-0.165 0.09 0.031" rpy=" 0 0 0"/>
-      <geometry>
-        <sphere radius="0.03"/>
-      </geometry>
-      <surface>
-        <friction>
-          <ode>
-            <mu>0</mu>
-            <mu2>0</mu2>
-            <slip1>1.0</slip1>
-            <slip2>1.0</slip2>
-          </ode>
-        </friction>
-      </surface>
-    </collision>
-    <visual name='caster_2_visual'>
-      <origin xyz="-0.165 0.09 0.031" rpy=" 0 0 0"/>
-      <geometry>
-        <sphere radius="0.03"/>
-      </geometry>
-    </visual>
-    <collision name='caster_3_collision'>
-      <origin xyz="0.165 -0.09 0.031" rpy=" 0 0 0"/>
-      <geometry>
-        <sphere radius="0.03"/>
-      </geometry>
-      <surface>
-        <friction>
-          <ode>
-            <mu>0</mu>
-            <mu2>0</mu2>
-            <slip1>1.0</slip1>
-            <slip2>1.0</slip2>
-          </ode>
-        </friction>
-      </surface>
-    </collision>
-    <visual name='caster_3_visual'>
-      <origin xyz="0.165 -0.09 0.031" rpy=" 0 0 0"/>
-      <geometry>
-        <sphere radius="0.03"/>
-      </geometry>
-    </visual>
-    <collision name='caster_4_collision'>
-      <origin xyz="-0.165 -0.09 0.031" rpy=" 0 0 0"/>
-      <geometry>
-        <sphere radius="0.03"/>
-      </geometry>
-      <surface>
-        <friction>
-          <ode>
-            <mu>0</mu>
-            <mu2>0</mu2>
-            <slip1>1.0</slip1>
-            <slip2>1.0</slip2>
-          </ode>
-        </friction>
-      </surface>
-    </collision>
-    <visual name='caster_4_visual'>
-      <origin xyz="-0.165 -0.09 0.031" rpy=" 0 0 0"/>
-      <geometry>
-        <sphere radius="0.03"/>
-      </geometry>
-    </visual>
-  </link>
-  <link
-    name="right_wheel_link">
-    <gravity>1</gravity>
-    <inertial>
-      <origin
-        xyz="0 0 0"
-        rpy="0 0 0" />
+          rgba="0.792156862745098 0.819607843137255 0.933333333333333 1" />
+      </material>
+    </visual>
+    <collision>
+      <origin
+        xyz="0 0 0"
+        rpy="0 0 0" />
+      <geometry>
+      <mesh filename="package://service_robot/meshes/wheel_right_link.STL" />
+      </geometry>
+    </collision>
+    <inertial>
+      <origin
+        xyz="0 0 0" rpy="0 0 0" />
       <mass value="0.238183102723089" />
       <inertia
@@ -151,108 +124,65 @@
         izz="0.000429469050110622" />
     </inertial>
-    <visual>
-      <origin
-        xyz="0 0 0"
-        rpy="0 0 0" />
-      <geometry>
-        <mesh
-          filename="package://service_robot/meshes/right_wheel_link.STL" />
-      </geometry>
-      <material
-        name="">
-        <color
-          rgba="0.792156862745098 0.819607843137255 0.933333333333333 1" />
-      </material>
-    </visual>
-    <collision>
-      <origin
-        xyz="0 0 0"
-        rpy="0 0 0" />
-      <geometry>
-        <mesh
-          filename="package://service_robot/meshes/right_wheel_link.STL" />
-      </geometry>
-    </collision>
-  </link>
-  <joint
-    name="wheel_right_joint"
-    type="continuous">
-    <origin
-      xyz="0.0049293 -0.235 0.074053"
-      rpy="0 0 0" />
-    <parent
-      link="base_link" />
-    <child
-      link="right_wheel_link" />
-    <axis
-      xyz="0 1 0" />
-    <limit
-      effort="10000"
-      velocity="100" />
-    <dynamics
-      damping="1"
-      friction="1" />
-  </joint>
-  <link
-    name="left_wheel_link">
-    <gravity>1</gravity>
-    <inertial>
-      <origin
-        xyz="0 0 0"
-        rpy="0 0 0" />
-      <mass
-        value="0.238183102723088" />
-      <inertia
-        ixx="0.000429468568590385"
-        ixy="2.82194133801453E-08"
-        ixz="3.45307405175469E-09"
-        iyy="0.000813895351440581"
-        iyz="9.00820636504668E-09"
-        izz="0.000429448713932949" />
-    </inertial>
-    <visual>
-      <origin
-        xyz="0 0 0"
-        rpy="0 0 0" />
-      <geometry>
-        <mesh
-          filename="package://service_robot/meshes/left_wheel_link.STL" />
-      </geometry>
-      <material
-        name="">
-        <color
-          rgba="0 0 0 1" />
-      </material>
-    </visual>
-    <collision>
-      <origin
-        xyz="0 0 0"
-        rpy="0 0 0" />
-      <geometry>
-        <mesh
-          filename="package://service_robot/meshes/left_wheel_link.STL" />
-      </geometry>
-    </collision>
-  </link>
-  <joint
-    name="wheel_left_joint"
-    type="continuous">
-    <origin
-      xyz="0.0047501 0.241 0.073998"
-      rpy="0 0 0" />
-    <parent
-      link="base_link" />
-    <child
-      link="left_wheel_link" />
-    <axis
-      xyz="0 1 0" />
-    <limit
-      effort="10000"
-      velocity="100" />
-    <dynamics
-      damping="1"
-      friction="1" />
-  </joint>
-  <link
+  </link>
+<!-- End wheel_right_link -->
+  <joint name="caster_1_joint" type="fixed">
+    <parent link="base_link"/>
+    <child link="caster_1"/>
+    <origin xyz="0.165 0.09 0.031" rpy="0 0 0"/>
+  </joint>
+  <link name="caster_1">
+    <collision>
+      <origin xyz="0.0 0.0 0.0" rpy=" 0 0 0"/>
+      <geometry>
+        <sphere radius="0.03"/>
+      </geometry>
+    </collision>
+  </link>
+  <joint name="caster_2_joint" type="fixed">
+    <parent link="base_link"/>
+    <child link="caster_2"/>
+    <origin xyz="-0.165 0.09 0.031" rpy="0 0 0"/>
+  </joint>
+  <link name="caster_2">
+    <collision>
+      <origin xyz="0.0 0.0 0.0" rpy=" 0 0 0"/>
+      <geometry>
+        <sphere radius="0.03"/>
+      </geometry>
+    </collision>
+  </link>
+  <joint name="caster_3_joint" type="fixed">
+    <parent link="base_link"/>
+    <child link="caster_3"/>
+    <origin xyz="0.165 -0.09 0.031" rpy="0 0 0"/>
+  </joint>
+  <link name="caster_3">
+    <collision>
+      <origin xyz="0.0 0.0 0.0" rpy=" 0 0 0"/>
+      <geometry>
+        <sphere radius="0.03"/>
+      </geometry>
+    </collision>
+  </link>
+   <joint name="caster_4_joint" type="fixed">
+    <parent link="base_link"/>
+    <child link="caster_4"/>
+    <origin xyz="-0.165 -0.09 0.031" rpy="0 0 0"/>
+  </joint>
+  <link name="caster_4">
+    <collision>
+      <origin xyz="0.0 0.0 0.0" rpy=" 0 0 0"/>
+      <geometry>
+        <sphere radius="0.03"/>
+      </geometry>
+    </collision>
+  </link>
+    <joint name="imu_joint" type="fixed">
+    <parent link="base_link"/>
+    <child link="imu_link"/>
+    <origin xyz="0 0 0" rpy="0 0 0"/>
+  </joint>
+  <link name="imu_link"/>
+ <link
     name="cloud">
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
Commit message: Add publish_planner_path.cpp

File: turtlebot3_description/urdf/mybot.xacro (robot description, xacro)
@@ -27,5 +27,5 @@
         rpy="0 0 0" />
       <geometry>
-      <mesh filename="package://service_robot/meshes/base_link.STL" />
+	<cylinder length="1.238" radius="0.25"/>
       </geometry>
     </collision>
@@ -64,5 +64,6 @@
       <origin xyz="0 0 0" rpy="0 0 0" />
       <geometry>
-      <mesh filename="package://service_robot/meshes/wheel_left_link.STL" />
+      <!--mesh filename="package://service_robot/meshes/wheel_left_link.STL" /-->
+      <cylinder length="0.033" radius="0.072"/>
       </geometry>
     </collision>
@@ -109,5 +110,5 @@
         rpy="0 0 0" />
       <geometry>
-      <mesh filename="package://service_robot/meshes/wheel_right_link.STL" />
+	<cylinder length="0.033" radius="0.072"/>
       </geometry>
     </collision>
@@ -185,5 +186,5 @@
   <link name="imu_link"/>
  <link
-    name="cloud">
+    name="base_scan">
     <inertial>
       <origin
@@ -233,5 +234,5 @@
       link="base_link" />
     <child
-      link="cloud" />
+      link="base_scan" />
     <axis
       xyz="0 0 0" />

Commit message: update

File: turtlebot3_description/urdf/mybot.xacro (robot description, xacro)
@@ -27,5 +27,5 @@
         rpy="0 0 0" />
       <geometry>
-	<cylinder length="1.238" radius="0.25"/>
+	<mesh filename="package://service_robot/meshes/base_link.STL" />
       </geometry>
     </collision>
@@ -64,6 +64,5 @@
       <origin xyz="0 0 0" rpy="0 0 0" />
       <geometry>
-      <!--mesh filename="package://service_robot/meshes/wheel_left_link.STL" /-->
-      <cylinder length="0.033" radius="0.072"/>
+      <mesh filename="package://service_robot/meshes/wheel_left_link.STL" />
       </geometry>
     </collision>
@@ -110,5 +109,5 @@
         rpy="0 0 0" />
       <geometry>
-	<cylinder length="0.033" radius="0.072"/>
+	<mesh filename="package://service_robot/meshes/wheel_right_link.STL" />
       </geometry>
     </collision>
